File: brama.sch (EAGLE design)
At the start: 64 parts, among them IC1 AT90USB162A, IC3 7806DT, J1 AVR_SPI_PRG_6OFFSET_PADS

Commit message: poprawki
Parts:
- removed J1: AVR_SPI_PRG_6OFFSET_PADS, SparkFun-Connectors:AVR_SPI_PRG_6OFFSET_PADS
- added C11: 100n, rcl:C-EUC0805
- added IC4: (no value), SparkFun-PowerIC:V_REG_LM1117SOT223
- added R21, R22: (no value), rcl:R-EU_R0805
Connections:
- removed net MISO: IC1.PB3(PDO/MISO), J1.1
- removed net MOSI: IC1.PB2(PDI/MISO), J1.4
- removed net SCK: IC1.PB1(SCK), J1.3
- new net N$33: IC4.ADJ, R21.1, R22.2
- new net UCAP: C1.2, IC1.UCAP
- net 3V3: now also C11.1, IC1.AVCC, IC4.OUT, IC4.OUT@1, R21.2; no longer C1.2, IC1.UCAP
- net 5V: now also IC4.IN; no longer J1.2
- net GND: now also C11.2, R22.1; no longer IC1.PD4(XCK/T0), J1.6
- net RESET: no longer J1.5
Changed lines of the file:
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@@
 <part name="GND8" library="SparkFun-Aesthetics" deviceset="GND" device=""/>
 <part name="GND9" library="SparkFun-Aesthetics" deviceset="GND" device=""/>
-<part name="J1" library="SparkFun-Connectors" deviceset="AVR_SPI_PRG_6" device="OFFSET_PADS"/>
-<part name="GND10" library="SparkFun-Aesthetics" deviceset="GND" device=""/>
 <part name="PHONE" library="SparkFun-Connectors" deviceset="M04" device="LONGPADS"/>
 <part name="GND11" library="SparkFun-Aesthetics" deviceset="GND" device=""/>
@@
 <part name="GND14" library="SparkFun-Aesthetics" deviceset="GND" device=""/>
 <part name="FRAME1" library="frames" deviceset="A3L-LOC" device=""/>
-<part name="GND15" library="SparkFun-Aesthetics" deviceset="GND" device=""/>
 <part name="JP2" library="SparkFun-Connectors" deviceset="M01" device="PTH"/>
 <part name="JP3" library="SparkFun-Connectors" deviceset="M01" device="PTH"/>
@@
 <part name="GND24" library="SparkFun-Aesthetics" deviceset="GND" device=""/>
 <part name="GND25" library="SparkFun-Aesthetics" deviceset="GND" device=""/>
+<part name="IC4" library="SparkFun-PowerIC" deviceset="V_REG_LM1117" device="SOT223"/>
+<part name="R21" library="rcl" deviceset="R-EU_" device="R0805"/>
+<part name="R22" library="rcl" deviceset="R-EU_" device="R0805"/>
+<part name="GND10" library="SparkFun-Aesthetics" deviceset="GND" device=""/>
+<part name="C11" library="rcl" deviceset="C-EU" device="C0805" value="100n"/>
+<part name="GND26" library="SparkFun-Aesthetics" deviceset="GND" device=""/>
 </parts>
 <sheets>
@@
 <instance part="GND8" gate="1" x="93.98" y="73.66"/>
 <instance part="GND9" gate="1" x="119.38" y="73.66"/>
-<instance part="J1" gate="G$1" x="177.8" y="220.98"/>
-<instance part="GND10" gate="1" x="190.5" y="213.36"/>
 <instance part="PHONE" gate="G$1" x="231.14" y="205.74" rot="R90"/>
 <instance part="GND11" gate="1" x="231.14" y="218.44" rot="R180"/>
@@
 <instance part="GND14" gate="1" x="177.8" y="101.6"/>
 <instance part="FRAME1" gate="G$1" x="0" y="0"/>
-<instance part="GND15" gate="1" x="121.92" y="170.18"/>
 <instance part="JP2" gate="G$1" x="208.28" y="152.4" rot="R90"/>
 <instance part="JP3" gate="G$1" x="132.08" y="86.36" rot="R90"/>
@@
 <instance part="GND24" gate="1" x="251.46" y="147.32"/>
 <instance part="GND25" gate="1" x="251.46" y="162.56" rot="R180"/>
+<instance part="IC4" gate="G$1" x="292.1" y="231.14"/>
+<instance part="R21" gate="G$1" x="302.26" y="220.98" rot="R90"/>
+<instance part="R22" gate="G$1" x="302.26" y="208.28" rot="R90"/>
+<instance part="GND10" gate="1" x="302.26" y="198.12"/>
+<instance part="C11" gate="G$1" x="307.34" y="228.6"/>
+<instance part="GND26" gate="1" x="307.34" y="220.98"/>
 </instances>
 <busses>
@@
 <wire x1="55.88" y1="228.6" x2="55.88" y2="231.14" width="0.1524" layer="91"/>
 <junction x="55.88" y="228.6"/>
-</segment>
-<segment>
-<pinref part="IC1" gate="G$1" pin="UCAP"/>
-<wire x1="58.42" y1="203.2" x2="43.18" y2="203.2" width="0.1524" layer="91"/>
-<pinref part="C1" gate="G$1" pin="2"/>
-<wire x1="43.18" y1="203.2" x2="40.64" y2="203.2" width="0.1524" layer="91"/>
-<wire x1="43.18" y1="200.66" x2="43.18" y2="203.2" width="0.1524" layer="91"/>
-<junction x="43.18" y="203.2"/>
-<label x="40.64" y="203.2" size="1.27" layer="95" rot="R180" xref="yes"/>
+<pinref part="IC1" gate="G$1" pin="AVCC"/>
+<wire x1="58.42" y1="218.44" x2="55.88" y2="218.44" width="0.1524" layer="91"/>
+<wire x1="55.88" y1="218.44" x2="55.88" y2="223.52" width="0.1524" layer="91"/>
+<junction x="55.88" y="223.52"/>
 </segment>
 <segment>
@@
 <wire x1="93.98" y1="104.14" x2="93.98" y2="106.68" width="0.1524" layer="91"/>
 <label x="93.98" y="106.68" size="1.27" layer="95" rot="R90" xref="yes"/>
+</segment>
+<segment>
+<pinref part="IC4" gate="G$1" pin="OUT@1"/>
+<pinref part="IC4" gate="G$1" pin="OUT"/>
+<wire x1="299.72" y1="228.6" x2="299.72" y2="231.14" width="0.1524" layer="91"/>
+<wire x1="299.72" y1="231.14" x2="302.26" y2="231.14" width="0.1524" layer="91"/>
+<pinref part="R21" gate="G$1" pin="2"/>
+<wire x1="302.26" y1="226.06" x2="302.26" y2="231.14" width="0.1524" layer="91"/>
+<wire x1="302.26" y1="231.14" x2="307.34" y2="231.14" width="0.1524" layer="91"/>
+<junction x="302.26" y="231.14"/>
+<junction x="299.72" y="231.14"/>
+<pinref part="C11" gate="G$1" pin="1"/>
+<label x="307.34" y="231.14" size="1.27" layer="95" rot="R90" xref="yes"/>
 </segment>
 </net>
@@
 </segment>
 <segment>
-<pinref part="J1" gate="G$1" pin="6"/>
-<wire x1="187.96" y1="218.44" x2="190.5" y2="218.44" width="0.1524" layer="91"/>
-<wire x1="190.5" y1="218.44" x2="190.5" y2="215.9" width="0.1524" layer="91"/>
-<pinref part="GND10" gate="1" pin="GND"/>
-</segment>
-<segment>
 <pinref part="PHONE" gate="G$1" pin="2"/>
 <wire x1="231.14" y1="210.82" x2="231.14" y2="215.9" width="0.1524" layer="91"/>
@@
 <pinref part="C6" gate="G$1" pin="2"/>
 <pinref part="GND14" gate="1" pin="GND"/>
-</segment>
-<segment>
-<pinref part="IC1" gate="G$1" pin="PD4(XCK/T0)"/>
-<wire x1="106.68" y1="175.26" x2="121.92" y2="175.26" width="0.1524" layer="91"/>
-<wire x1="121.92" y1="175.26" x2="121.92" y2="172.72" width="0.1524" layer="91"/>
-<pinref part="GND15" gate="1" pin="GND"/>
 </segment>
 <segment>
@@
 <pinref part="GND25" gate="1" pin="GND"/>
 </segment>
+<segment>
+<pinref part="GND10" gate="1" pin="GND"/>
+<pinref part="R22" gate="G$1" pin="1"/>
+<wire x1="302.26" y1="200.66" x2="302.26" y2="203.2" width="0.1524" layer="91"/>
+</segment>
+<segment>
+<pinref part="C11" gate="G$1" pin="2"/>
+<pinref part="GND26" gate="1" pin="GND"/>
+</segment>
 </net>
 <net name="5V" class="0">
@@
 <wire x1="58.42" y1="220.98" x2="48.26" y2="220.98" width="0.1524" layer="91"/>
 <label x="48.26" y="220.98" size="1.27" layer="95" rot="R180" xref="yes"/>
-</segment>
-<segment>
-<pinref part="J1" gate="G$1" pin="2"/>
-<wire x1="187.96" y1="223.52" x2="193.04" y2="223.52" width="0.1524" layer="91"/>
-<label x="193.04" y="223.52" size="1.27" layer="95" xref="yes"/>
 </segment>
 <segment>
@@
 <junction x="231.14" y="175.26"/>
 </segment>
+<segment>
+<pinref part="IC4" gate="G$1" pin="IN"/>
+<wire x1="284.48" y1="231.14" x2="281.94" y2="231.14" width="0.1524" layer="91"/>
+<label x="281.94" y="231.14" size="1.27" layer="95" rot="R180" xref="yes"/>
+</segment>
 </net>
 <net name="RESET" class="0">
@@
 <junction x="35.56" y="177.8"/>
 <label x="27.94" y="177.8" size="1.27" layer="95" rot="R180" xref="yes"/>
-</segment>
-<segment>
-<pinref part="J1" gate="G$1" pin="5"/>
-<wire x1="170.18" y1="218.44" x2="165.1" y2="218.44" width="0.1524" layer="91"/>
-<label x="165.1" y="218.44" size="1.27" layer="95" rot="R180" xref="yes"/>
 </segment>
 </net>
@@
 <wire x1="106.68" y1="203.2" x2="111.76" y2="203.2" width="0.1524" layer="91"/>
 <label x="111.76" y="203.2" size="1.27" layer="95" xref="yes"/>
-</segment>
-</net>
-<net name="MOSI" class="0">
-<segment>
-<pinref part="IC1" gate="G$1" pin="PB2(PDI/MISO)"/>
-<wire x1="106.68" y1="193.04" x2="111.76" y2="193.04" width="0.1524" layer="91"/>
-<label x="111.76" y="193.04" size="1.27" layer="95" xref="yes"/>
-</segment>
-<segment>
-<pinref part="J1" gate="G$1" pin="4"/>
-<wire x1="187.96" y1="220.98" x2="193.04" y2="220.98" width="0.1524" layer="91"/>
-<label x="193.04" y="220.98" size="1.27" layer="95" xref="yes"/>
-</segment>
-</net>
-<net name="MISO" class="0">
-<segment>
-<pinref part="IC1" gate="G$1" pin="PB3(PDO/MISO)"/>
-<wire x1="106.68" y1="195.58" x2="111.76" y2="195.58" width="0.1524" layer="91"/>
-<label x="111.76" y="195.58" size="1.27" layer="95" xref="yes"/>
-</segment>
-<segment>
-<pinref part="J1" gate="G$1" pin="1"/>
-<wire x1="170.18" y1="223.52" x2="165.1" y2="223.52" width="0.1524" layer="91"/>
-<label x="165.1" y="223.52" size="1.27" layer="95" rot="R180" xref="yes"/>
-</segment>
-</net>
-<net name="SCK" class="0">
-<segment>
-<pinref part="IC1" gate="G$1" pin="PB1(SCK)"/>
-<wire x1="106.68" y1="190.5" x2="111.76" y2="190.5" width="0.1524" layer="91"/>
-<label x="111.76" y="190.5" size="1.27" layer="95" xref="yes"/>
-</segment>
-<segment>
-<pinref part="J1" gate="G$1" pin="3"/>
-<wire x1="170.18" y1="220.98" x2="165.1" y2="220.98" width="0.1524" layer="91"/>
-<label x="165.1" y="220.98" size="1.27" layer="95" rot="R180" xref="yes"/>
 </segment>
 </net>
@@
 </segment>
 </net>
+<net name="N$33" class="0">
+<segment>
+<pinref part="R21" gate="G$1" pin="1"/>
+<pinref part="R22" gate="G$1" pin="2"/>
+<wire x1="302.26" y1="215.9" x2="302.26" y2="213.36" width="0.1524" layer="91"/>
+<pinref part="IC4" gate="G$1" pin="ADJ"/>
+<wire x1="292.1" y1="223.52" x2="292.1" y2="215.9" width="0.1524" layer="91"/>
+<wire x1="292.1" y1="215.9" x2="302.26" y2="215.9" width="0.1524" layer="91"/>
+<junction x="302.26" y="215.9"/>
+</segment>
+</net>
+<net name="UCAP" class="0">
+<segment>
+<pinref part="IC1" gate="G$1" pin="UCAP"/>
+<wire x1="58.42" y1="203.2" x2="43.18" y2="203.2" width="0.1524" layer="91"/>
+<pinref part="C1" gate="G$1" pin="2"/>
+<wire x1="43.18" y1="200.66" x2="43.18" y2="203.2" width="0.1524" layer="91"/>
+</segment>
+</net>
