File: brama.brd (EAGLE design)
At the start: 92.7 x 127.5 mm, 68 parts, among them IC1 AT90USB162A, IC3 7806DT, J1 AVR_SPI_PRG_6OFFSET_PADS

Commit message: poprawki
Parts:
- removed J1: AVR_SPI_PRG_6OFFSET_PADS, SparkFun-Connectors:2X3_OFFSET
- added C11: 100n, rcl:C0805
- added IC4: (no value), SparkFun-PowerIC:SOT223
- added R21, R22: (no value), rcl:R0805
- moved C5 34.5 mm to (35.3, 79.9), turned to 270 degrees
- moved C7 24.6 mm to (32.2, 101.2), turned to 90 degrees
- moved U$6 20.0 mm to (36.2, 101.8), turned to 270 degrees
- moved R19 18.7 mm to (35.2, 97.4), turned to 90 degrees
- moved L1 18.1 mm to (39.8, 103.8), turned to 270 degrees
- moved R20 16.2 mm to (3.81, 96.7), turned to 0 degrees
- moved R18 15.7 mm to (37.6, 97.7), turned to 270 degrees
- moved C8 12.7 mm to (39.9, 97.7), turned to 90 degrees
- moved C10 12.5 mm to (10.4, 39.0)
- moved C9 12.5 mm to (4.53, 37.8)
- moved IC3 12.5 mm to (9.67, 30.7)
- moved JP10 12.5 mm to (4.59, 23.4)
- moved JP9 12.5 mm to (4.59, 14.5)
- moved D1 10.7 mm to (43.1, 99.8), turned to 90 degrees
- moved JP8 4.44 mm to (47.6, 97.1), turned to 270 degrees
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Connections:
- removed net MISO: IC1.17, J1.1
- removed net MOSI: IC1.16, J1.4
- removed net SCK: IC1.15, J1.3
- new net N$33: IC4.1, R21.1, R22.2
- new net UCAP: C1.2, IC1.27
- net 3V3: now also C11.1, IC1.32, IC4.2, IC4.4, R21.2; no longer C1.2, IC1.27
- net 5V: now also IC4.3; no longer J1.2
- net GND: now also C11.2, R22.1; no longer IC1.10, J1.6
- net RESET: no longer J1.5
Routing:
- net RESET: track 57.4 -> 8.89 mm
- net 5V: track 314.5 -> 357.2 mm
- net 3V3: track 150.6 -> 124.0 mm
- net N$33: track 0.00 -> 14.0 mm
- net MISO: track 13.9 -> 0.00 mm
- net SCK: track 12.8 -> 0.00 mm
- net MOSI: track 9.57 -> 0.00 mm
- net GND: track 11.9 -> 3.31 mm
- net UCAP: track 0.00 -> 6.86 mm
- net D-: track 3.20 -> 9.58 mm
- net N$1: track 11.5 -> 6.07 mm
- net 12V: track 72.2 -> 76.7 mm
- net RXD: track 50.5 -> 46.9 mm
- net D+: track 3.99 -> 4.93 mm
- net VIN: track 17.0 -> 16.2 mm
Other:
- board size 92.7 x 127.5 mm -> 95 x 127.5 mm

Commit message: piszemy soft
Parts:
- moved JP2 1.27 mm to (30.1, 111.8)
Changed lines of the file:
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@@
 <setting verticaltext="up"/>
 </settings>
-<grid distance="0" unitdist="inch" unit="inch" style="lines" multiple="1" display="yes" altdistance="0.003937" altunitdist="inch" altunit="inch"/>
+<grid distance="0.05" unitdist="inch" unit="inch" style="lines" multiple="1" display="yes" altdistance="0.025" altunitdist="inch" altunit="inch"/>
 <layers>
 <layer number="1" name="Top" color="4" fill="1" visible="yes" active="yes"/>
@@
 <element name="R17" library="rcl" package="R0805" value="" x="34.671" y="118.11" rot="MR180"/>
 <element name="C6" library="rcl" package="C0805" value="100n" x="67.945" y="121.285" rot="MR0"/>
-<element name="JP2" library="SparkFun-Connectors" package="1X01" value="M01PTH" x="30.099" y="113.03"/>
+<element name="JP2" library="SparkFun-Connectors" package="1X01" value="M01PTH" x="30.099" y="111.76"/>
 <element name="JP3" library="SparkFun-Connectors" package="1X01" value="M01PTH" x="12.7" y="77.47"/>
 <element name="JP4" library="SparkFun-Connectors" package="1X01" value="M01PTH" x="10.033" y="77.47"/>
@@
 <wire x1="24.13" y1="108.5026" x2="24.13" y2="109.601" width="0.4064" layer="16"/>
 <wire x1="24.13" y1="109.601" x2="25.527" y2="110.998" width="0.4064" layer="16"/>
-<wire x1="25.527" y1="110.998" x2="30.099" y2="113.03" width="0.4064" layer="16"/>
+<wire x1="25.527" y1="110.998" x2="30.099" y2="111.76" width="0.4064" layer="16"/>
 </signal>
 <signal name="GATE">
